File: Pico-Skidi.kicad_sch (KiCad schematic)
At the start: 1 part, among them SW1 BOOTSEL

Commit message: syncing
Parts:
- removed SW1: BOOTSEL, symbol Switch:SW_SPST
Changed lines of the file:
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@@
-    (stroke (width 0) (type default))
-  )
-  (wire (pts (xy 102.87 34.29) (xy 102.87 46.99))
     (stroke (width 0) (type default))
   )
@@
     (stroke (width 0) (type default))
   )
-  (wire (pts (xy 123.19 46.99) (xy 119.38 46.99))
-    (stroke (width 0) (type default))
-  )
-  (wire (pts (xy 97.79 34.29) (xy 102.87 34.29))
-    (stroke (width 0) (type default))
-  )
   (wire (pts (xy 52.07 19.05) (xy 68.58 19.05))
     (stroke (width 0) (type default))
@@
     (stroke (width 0) (type default))
   )
-  (wire (pts (xy 102.87 46.99) (xy 109.22 46.99))
-    (stroke (width 0) (type default))
-  )
   (wire (pts (xy 97.79 31.75) (xy 106.68 31.75))
     (stroke (width 0) (type default))
@@
     )
   )
-  (symbol (lib_id "Switch:SW_SPST") (at 114.3 46.99 0) (unit 1)
-    (in_bom yes) (on_board yes) (dnp no) (fields_autoplaced)
-    (property "Reference" "SW1" (at 114.3 40.64 0)
-      (effects (font (size 1.27 1.27)))
-    )
-    (property "Value" "BOOTSEL" (at 114.3 43.18 0)
-      (effects (font (size 1.27 1.27)))
-    )
-    (property "Footprint" "" (at 114.3 46.99 0)
-      (effects (font (size 1.27 1.27)) hide)
-    )
-    (property "Datasheet" "~" (at 114.3 46.99 0)
-      (effects (font (size 1.27 1.27)) hide)
-    )
-    (pin "1")
-    (pin "2")
-    (instances
-      (project "Pico-Skidi"
-        (path "/21865b85-eb74-4d61-a31a-30858d3bc341"
-          (reference "SW1") (unit 1)
-        )
-      )
-    )
-  )
   (symbol (lib_id "power:PWR_FLAG") (at 22.86 96.52 0) (unit 1)
     (in_bom yes) (on_board yes) (dnp no) (fields_autoplaced)
@@
   (symbol (lib_id "power:+5V") (at 30.48 96.52 0) (unit 1)
     (in_bom yes) (on_board yes) (dnp no) (fields_autoplaced)
-    (property "Reference" "#PWR050" (at 30.48 100.33 0)
+    (property "Reference" "#PWR02" (at 30.48 100.33 0)
       (effects (font (size 1.27 1.27)) hide)
     )
@@
       (project "Pico-Skidi"
         (path "/21865b85-eb74-4d61-a31a-30858d3bc341"
-          (reference "#PWR050") (unit 1)
+          (reference "#PWR02") (unit 1)
         )
       )
@@
   (symbol (lib_id "power:VBUS") (at 50.8 96.52 0) (unit 1)
     (in_bom yes) (on_board yes) (dnp no) (fields_autoplaced)
-    (property "Reference" "#PWR052" (at 50.8 100.33 0)
+    (property "Reference" "#PWR04" (at 50.8 100.33 0)
       (effects (font (size 1.27 1.27)) hide)
     )
@@
       (project "Pico-Skidi"
         (path "/21865b85-eb74-4d61-a31a-30858d3bc341"
-          (reference "#PWR052") (unit 1)
-        )
-      )
-    )
-  )
-  (symbol (lib_id "power:GND") (at 123.19 46.99 0) (unit 1)
-    (in_bom yes) (on_board yes) (dnp no) (fields_autoplaced)
-    (property "Reference" "#PWR01" (at 123.19 53.34 0)
-      (effects (font (size 1.27 1.27)) hide)
-    )
-    (property "Value" "GND" (at 123.19 52.07 0)
-      (effects (font (size 1.27 1.27)))
-    )
-    (property "Footprint" "" (at 123.19 46.99 0)
-      (effects (font (size 1.27 1.27)) hide)
-    )
-    (property "Datasheet" "" (at 123.19 46.99 0)
+          (reference "#PWR04") (unit 1)
+        )
+      )
+    )
+  )
+  (symbol (lib_id "power:GND") (at 22.86 96.52 0) (unit 1)
+    (in_bom yes) (on_board yes) (dnp no) (fields_autoplaced)
+    (property "Reference" "#PWR01" (at 22.86 102.87 0)
+      (effects (font (size 1.27 1.27)) hide)
+    )
+    (property "Value" "GND" (at 22.86 101.6 0)
+      (effects (font (size 1.27 1.27)))
+    )
+    (property "Footprint" "" (at 22.86 96.52 0)
+      (effects (font (size 1.27 1.27)) hide)
+    )
+    (property "Datasheet" "" (at 22.86 96.52 0)
       (effects (font (size 1.27 1.27)) hide)
     )
@@
     )
   )
-  (symbol (lib_id "power:GND") (at 22.86 96.52 0) (unit 1)
-    (in_bom yes) (on_board yes) (dnp no) (fields_autoplaced)
-    (property "Reference" "#PWR049" (at 22.86 102.87 0)
-      (effects (font (size 1.27 1.27)) hide)
-    )
-    (property "Value" "GND" (at 22.86 101.6 0)
-      (effects (font (size 1.27 1.27)))
-    )
-    (property "Footprint" "" (at 22.86 96.52 0)
-      (effects (font (size 1.27 1.27)) hide)
-    )
-    (property "Datasheet" "" (at 22.86 96.52 0)
-      (effects (font (size 1.27 1.27)) hide)
-    )
-    (pin "1")
-    (instances
-      (project "Pico-Skidi"
-        (path "/21865b85-eb74-4d61-a31a-30858d3bc341"
-          (reference "#PWR049") (unit 1)
-        )
-      )
-    )
-  )
   (symbol (lib_id "power:+3.3V") (at 40.64 96.52 0) (unit 1)
     (in_bom yes) (on_board yes) (dnp no) (fields_autoplaced)
-    (property "Reference" "#PWR051" (at 40.64 100.33 0)
+    (property "Reference" "#PWR03" (at 40.64 100.33 0)
       (effects (font (size 1.27 1.27)) hide)
     )
@@
       (project "Pico-Skidi"
         (path "/21865b85-eb74-4d61-a31a-30858d3bc341"
-          (reference "#PWR051") (unit 1)
-        )
-      )
+          (reference "#PWR03") (unit 1)
+        )
+      )

Commit message: progress at last
Other:
- removed sheet Power Management
Changed lines of the file:
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@@
 (kicad_sch (version 20230121) (generator eeschema)
   (paper "A4")
-  (junction (at 82.55 64.77) (diameter 0) (color 0 0 0 0)
-  )
-  (junction (at 82.55 62.23) (diameter 0) (color 0 0 0 0)
-  )
-  (wire (pts (xy 82.55 64.77) (xy 96.52 64.77))
-    (stroke (width 0) (type default))
-  )
   (wire (pts (xy 52.07 36.83) (xy 68.58 36.83))
     (stroke (width 0) (type default))
   )
-  (wire (pts (xy 93.98 45.72) (xy 93.98 62.23))
-    (stroke (width 0) (type default))
-  )
   (wire (pts (xy 52.07 31.75) (xy 68.58 31.75))
     (stroke (width 0) (type default))
@@
     (stroke (width 0) (type default))
   )
-  (wire (pts (xy 96.52 45.72) (xy 96.52 64.77))
-    (stroke (width 0) (type default))
-  )
   (wire (pts (xy 52.07 26.67) (xy 68.58 26.67))
     (stroke (width 0) (type default))
@@
     (stroke (width 0) (type default))
   )
-  (wire (pts (xy 82.55 62.23) (xy 93.98 62.23))
-    (stroke (width 0) (type default))
-  )
   (wire (pts (xy 55.88 60.96) (xy 39.37 60.96))
     (stroke (width 0) (type default))
@@
   )
   (wire (pts (xy 91.44 53.34) (xy 55.88 53.34))
-    (stroke (width 0) (type default))
-  )
-  (wire (pts (xy 82.55 64.77) (xy 82.55 62.23))
     (stroke (width 0) (type default))
   )
@@
       )
     )
-  )
-  (sheet (at 69.85 57.15) (size 12.7 10.16) (fields_autoplaced)
-    (stroke (width 0.1524) (type solid))
-    (fill (color 0 0 0 0.0000))
-    (property "Sheetname" "Power Management" (at 69.85 56.4384 0)
-      (effects (font (size 1.27 1.27)) (justify left bottom))
-    )
-    (property "Sheetfile" "Power.kicad_sch" (at 69.85 67.8946 0) (show_name)
-      (effects (font (size 1.27 1.27)) (justify left top))
-    )
-    (pin "D-" output (at 82.55 62.23 0)
-      (effects (font (size 1.27 1.27)) (justify right))
-    )
-    (pin "D+" output (at 82.55 64.77 0)
-      (effects (font (size 1.27 1.27)) (justify right))
-    )
-    (instances
-      (project "Pico-Skidi"
-        (path "/21865b85-eb74-4d61-a31a-30858d3bc341" (page "2"))
-      )
-    )
