File: Pico-Skidi.kicad_sch (KiCad schematic)
At the start: 0 parts

Commit message: Adding Power
Parts:
- added J1: Conn_01x02, Connector_JST:JST_PH_S2B-PH-SM4-TB_1x02-1MP_P2.00mm_Horizontal, symbol Connector_Generic:Conn_01x02
- added U1: ~, pico-skidi:TPS61023, symbol Pico-Skidi:TPS61023
- added U2: ~, pico-skidi:Pimoroni Amigo Pro Mounts, symbol Pico-Skidi:Pimoroni_Amigo_Pro
Connections:
- net +5V: now also U1.3 (5v)
- net GND: now also J1.2 (Pin_2), U1.2 (GND), U2.14 (DEV-)
- new net DEV+: J1.1 (Pin_1), U1.1 (VIN), U2.13 (DEV+)
- no-connect marks 0 -> 16
Other:
- sheet Pico W ports: added VSYS; removed USB_D+, USB_D-
