File: Motors.kicad_sch (KiCad schematic)
At the start: 5 parts, among them M1 Motor_DC, M2 Motor_DC, M3 Motor_DC, U2 PDRV8411PWPR, U3 PDRV8411PWPR

Commit message: Lots of changes
Parts:
- added C2, C3, C4, C5: C, Capacitor_SMD:C_0603_1608Metric_Pad1.08x0.95mm_HandSolder, symbol Device:C
- added J3, J4, J5, J6: Conn_01x02, Connector_PinHeader_2.54mm:PinHeader_1x02_P2.54mm_Vertical, symbol Connector_Generic:Conn_01x02
- added M3: Motor_DC, Motors:Vybronics_VZ30C1T8219732L, symbol Motor:Motor_DC
- added R6, R7, R8, R9: R, symbol Device:R
- M1, M2, M3: footprint (none) -> Motors:Vybronics_VZ30C1T8219732L
Connections:
- net GND: now also U2.EPAD, U3.EPAD, C2.2, C3.2, C4.2, C5.2, R6.2, R7.2, R8.2, R9.2
- net at U3.1 (AISEN): now also R6.1
- net +5V: now reaches U3.10 (VM)
- net +5V: now also U2.10 (VM), C2.1, C3.1, C4.1, C5.1
- net MOT_C-: now reaches U3.13 (AIN2)
- net MOT_C+: now reaches U3.14 (AIN1)
- net at U3.16 (AOUT1): now also M3.1 (+), J3.1 (Pin_1)
- net at U3.2 (AOUT2): now also M3.2 (-), J3.2 (Pin_2)
- net at U3.3 (BOUT2): now also J4.2 (Pin_2), M3.2 (-)
- net at U3.4 (BISEN): now also R8.1
- net at U3.5 (BOUT1): now also J4.1 (Pin_1), M3.1 (+)
- net nFAULT_02: now reaches U3.6 (nFAULT)
- net MOT_D+: now reaches U3.7 (BIN1)
- net MOT_D-: now reaches U3.8 (BIN2)
- net at U2.1 (AISEN): now also R7.1
- net MOT_A-: now reaches U2.13 (AIN2)
- net MOT_A+: now reaches U2.14 (AIN1)
- net at U2.16 (AOUT1): now also M1.1 (+), J5.1 (Pin_1)
- net at U2.2 (AOUT2): now also M1.2 (-), J5.2 (Pin_2)
- net at U2.3 (BOUT2): now also M2.2 (-), J6.2 (Pin_2)
- net at U2.4 (BISEN): now also R9.1
- net at U2.5 (BOUT1): now also M2.1 (+), J6.1 (Pin_1)
- net nFAULT_01: now reaches U2.6 (nFAULT)
- net MOT_B+: now reaches U2.7 (BIN1)
- net MOT_B-: now reaches U2.8 (BIN2)
- no-connect marks 0 -> 2
Other:
- moved on the sheet: M1, M2, M3

Commit message: syncing
Parts:
- removed M1, M2, M3 (x2): Motor_DC, Motors:Vybronics_VZ30C1T8219732L, symbol Motor:Motor_DC
- J3: value Conn_01x02 -> Motor 3
- J4: value Conn_01x02 -> Motor 4
- J5: value Conn_01x02 -> Motor 1
- J6: value Conn_01x02 -> Motor 2
- R10: renamed from R7; footprint (none) -> Resistor_SMD:R_0603_1608Metric_Pad0.98x0.95mm_HandSolder
- R11: renamed from R8; footprint (none) -> Resistor_SMD:R_0603_1608Metric_Pad0.98x0.95mm_HandSolder
- R12: renamed from R9; footprint (none) -> Resistor_SMD:R_0603_1608Metric_Pad0.98x0.95mm_HandSolder
- R9: renamed from R6; footprint (none) -> Resistor_SMD:R_0603_1608Metric_Pad0.98x0.95mm_HandSolder
- U2, U3: footprint TSSOP_11PWPR_TEX -> DRV8411:TSSOP_11PWPR_TEX
- renumbered C2 to C4, C3 to C5, C4 to C6, C5 to C7

Commit message: Adding Power
Parts:
- renumbered C4 to C1, C5 to C2, C6 to C3, C7 to C4, J3 to J2, J4 to J3, J5 to J4, J6 to J5, R9 to R1, R10 to R2, R11 to R3, R12 to R4
