File: PicoW.kicad_sch (KiCad schematic)
At the start: 3 parts, among them J7 Conn_01x03, J8 Conn_01x04, U1 Pico

Commit message: progress at last
Parts:
- removed J7: Conn_01x03, Connector_PinHeader_2.54mm:PinHeader_1x03_P2.54mm_Vertical, symbol Connector_Generic:Conn_01x03
- U1: footprint MCU_RaspberryPi_and_Boards:RPi_Pico_W_SMD -> pico-skidi:RPi_Pico_TH
Connections:
- net GND: no longer U1.42 (GND)
- net +5V renamed VSYS
- net USB_D+: no longer names the net of U1.45 (D+)
- net USB_D-: no longer names the net of U1.46 (D-)
- no-connect marks 9 -> 15
Changed lines of the file:
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@@
   (junction (at 168.91 110.49) (diameter 0) (color 0 0 0 0)
   )
-  (junction (at 142.24 128.27) (diameter 0) (color 0 0 0 0)
-  )
   (junction (at 111.76 85.09) (diameter 0) (color 0 0 0 0)
   )
@@
   (junction (at 111.76 110.49) (diameter 0) (color 0 0 0 0)
   )
+  (no_connect (at 144.78 120.65))
+  (no_connect (at 139.7 62.23))
+  (no_connect (at 140.97 95.25))
   (no_connect (at 160.02 80.01))
   (no_connect (at 160.02 95.25))
+  (no_connect (at 142.24 62.23))
   (no_connect (at 160.02 92.71))
   (no_connect (at 124.46 67.31))
   (no_connect (at 124.46 69.85))
+  (no_connect (at 139.7 120.65))
   (no_connect (at 160.02 74.93))
   (no_connect (at 160.02 102.87))
   (no_connect (at 124.46 115.57))
   (no_connect (at 160.02 82.55))
-  (wire (pts (xy 132.08 134.62) (xy 132.08 130.81))
-    (stroke (width 0) (type default))
-  )
+  (no_connect (at 142.24 120.65))
   (wire (pts (xy 137.16 62.23) (xy 137.16 58.42))
     (stroke (width 0) (type default))
@@
     (stroke (width 0) (type default))
   )
-  (wire (pts (xy 139.7 120.65) (xy 139.7 125.73))
-    (stroke (width 0) (type default))
-  )
   (wire (pts (xy 193.04 62.23) (xy 195.58 62.23))
     (stroke (width 0) (type default))
@@
     (stroke (width 0) (type default))
   )
-  (wire (pts (xy 144.78 120.65) (xy 144.78 134.62))
-    (stroke (width 0) (type default))
-  )
   (wire (pts (xy 163.83 78.74) (xy 163.83 77.47))
     (stroke (width 0) (type default))
@@
     (stroke (width 0) (type default))
   )
-  (wire (pts (xy 142.24 120.65) (xy 142.24 128.27))
-    (stroke (width 0) (type default))
-  )
   (wire (pts (xy 160.02 72.39) (xy 170.18 72.39))
     (stroke (width 0) (type default))
@@
     (stroke (width 0) (type default))
   )
-  (wire (pts (xy 142.24 128.27) (xy 132.08 128.27))
-    (stroke (width 0) (type default))
-  )
   (wire (pts (xy 165.1 67.31) (xy 160.02 67.31))
     (stroke (width 0) (type default))
@@
     (stroke (width 0) (type default))
   )
-  (wire (pts (xy 139.7 125.73) (xy 132.08 125.73))
-    (stroke (width 0) (type default))
-  )
   (wire (pts (xy 111.76 72.39) (xy 124.46 72.39))
     (stroke (width 0) (type default))
   )
   (wire (pts (xy 111.76 97.79) (xy 111.76 110.49))
-    (stroke (width 0) (type default))
-  )
-  (wire (pts (xy 144.78 134.62) (xy 132.08 134.62))
     (stroke (width 0) (type default))
   )
@@
     (effects (font (size 1.27 1.27)) (justify right))
   )
-  (hierarchical_label "USB_D-" (shape bidirectional) (at 142.24 62.23 90) (fields_autoplaced)
-    (effects (font (size 1.27 1.27)) (justify left))
-  )
   (hierarchical_label "BOOTSEL" (shape input) (at 149.86 62.23 90) (fields_autoplaced)
     (effects (font (size 1.27 1.27)) (justify left))
@@
   (hierarchical_label "nFAULT_01" (shape input) (at 124.46 100.33 180) (fields_autoplaced)
     (effects (font (size 1.27 1.27)) (justify right))
-  )
-  (hierarchical_label "USB_D+" (shape bidirectional) (at 139.7 62.23 90) (fields_autoplaced)
-    (effects (font (size 1.27 1.27)) (justify left))
   )
   (hierarchical_label "SRV_05" (shape output) (at 124.46 92.71 180) (fields_autoplaced)
@@
     )
   )
-  (symbol (lib_id "power:+5V") (at 171.45 69.85 0) (unit 1)
-    (in_bom yes) (on_board yes) (dnp no) (fields_autoplaced)
-    (property "Reference" "#PWR039" (at 171.45 73.66 0)
-      (effects (font (size 1.27 1.27)) hide)
-    )
-    (property "Value" "+5V" (at 171.45 64.77 0)
+  (symbol (lib_id "power:+3.3V") (at 187.96 68.58 0) (unit 1)
+    (in_bom yes) (on_board yes) (dnp no) (fields_autoplaced)
+    (property "Reference" "#PWR040" (at 187.96 72.39 0)
+      (effects (font (size 1.27 1.27)) hide)
+    )
+    (property "Value" "+3.3V" (at 187.96 63.5 0)
+      (effects (font (size 1.27 1.27)))
+    )
+    (property "Footprint" "" (at 187.96 68.58 0)
+      (effects (font (size 1.27 1.27)) hide)
+    )
+    (property "Datasheet" "" (at 187.96 68.58 0)
+      (effects (font (size 1.27 1.27)) hide)
+    )
+    (pin "1")
+    (instances
+      (project "Pico-Skidi"
+        (path "/21865b85-eb74-4d61-a31a-30858d3bc341/60530e3c-b075-4fd7-83a5-48bc65381cc4"
+          (reference "#PWR040") (unit 1)
+        )
+      )
+    )
+  )
+  (symbol (lib_id "power:VBUS") (at 165.1 67.31 0) (unit 1)
+    (in_bom yes) (on_board yes) (dnp no) (fields_autoplaced)
+    (property "Reference" "#PWR036" (at 165.1 71.12 0)
+      (effects (font (size 1.27 1.27)) hide)
+    )
+    (property "Value" "VBUS" (at 165.1 62.23 0)
+      (effects (font (size 1.27 1.27)))
+    )
+    (property "Footprint" "" (at 165.1 67.31 0)
+      (effects (font (size 1.27 1.27)) hide)
+    )
+    (property "Datasheet" "" (at 165.1 67.31 0)
+      (effects (font (size 1.27 1.27)) hide)
+    )
+    (pin "1")
+    (instances
+      (project "Pico-Skidi"
+        (path "/21865b85-eb74-4d61-a31a-30858d3bc341/60530e3c-b075-4fd7-83a5-48bc65381cc4"
+          (reference "#PWR036") (unit 1)
+        )
+      )
+    )
+  )
+  (symbol (lib_id "ExtraPower:VSYS") (at 171.45 69.85 0) (unit 1)
+    (in_bom yes) (on_board yes) (dnp no) (fields_autoplaced)
+    (property "Reference" "#PWR05" (at 171.45 73.66 0)
+      (effects (font (size 1.27 1.27)) hide)
+    )
+    (property "Value" "VSYS" (at 171.45 64.77 0)
       (effects (font (size 1.27 1.27)))
     )
@@
       (project "Pico-Skidi"
         (path "/21865b85-eb74-4d61-a31a-30858d3bc341/60530e3c-b075-4fd7-83a5-48bc65381cc4"
-          (reference "#PWR039") (unit 1)
-        )
-      )
-    )
-  )
-  (symbol (lib_id "power:+3.3V") (at 187.96 68.58 0) (unit 1)
-    (in_bom yes) (on_board yes) (dnp no) (fields_autoplaced)
-    (property "Reference" "#PWR040" (at 187.96 72.39 0)
-      (effects (font (size 1.27 1.27)) hide)
-    )
-    (property "Value" "+3.3V" (at 187.96 63.5 0)
-      (effects (font (size 1.27 1.27)))
-    )
-    (property "Footprint" "" (at 187.96 68.58 0)
-      (effects (font (size 1.27 1.27)) hide)
-    )
-    (property "Datasheet" "" (at 187.96 68.58 0)
-      (effects (font (size 1.27 1.27)) hide)
-    )
-    (pin "1")
-    (instances
-      (project "Pico-Skidi"
-        (path "/21865b85-eb74-4d61-a31a-30858d3bc341/60530e3c-b075-4fd7-83a5-48bc65381cc4"
-          (reference "#PWR040") (unit 1)
-        )
-      )
-    )
-  )
-  (symbol (lib_id "power:VBUS") (at 165.1 67.31 0) (unit 1)
-    (in_bom yes) (on_board yes) (dnp no) (fields_autoplaced)
-    (property "Reference" "#PWR036" (at 165.1 71.12 0)
-      (effects (font (size 1.27 1.27)) hide)
-    )
-    (property "Value" "VBUS" (at 165.1 62.23 0)
-      (effects (font (size 1.27 1.27)))
-    )
-    (property "Footprint" "" (at 165.1 67.31 0)
-      (effects (font (size 1.27 1.27)) hide)
-    )
-    (property "Datasheet" "" (at 165.1 67.31 0)
-      (effects (font (size 1.27 1.27)) hide)
-    )
-    (pin "1")
-    (instances
-      (project "Pico-Skidi"
-        (path "/21865b85-eb74-4d61-a31a-30858d3bc341/60530e3c-b075-4fd7-83a5-48bc65381cc4"
-          (reference "#PWR036") (unit 1)
+          (reference "#PWR05") (unit 1)
         )
       )
@@
       (effects (font (size 1.27 1.27)))
     )
-    (property "Footprint" "MCU_RaspberryPi_and_Boards:RPi_Pico_W_SMD" (at 142.24 91.44 90)
+    (property "Footprint" "pico-skidi:RPi_Pico_TH" (at 142.24 91.44 90)
       (effects (font (size 1.27 1.27)) hide)
     )
@@
         )
       )
-    )
-  )
-  (symbol (lib_id "power:GND") (at 142.24 128.27 0) (unit 1)
-    (in_bom yes) (on_board yes) (dnp no) (fields_autoplaced)
-    (property "Reference" "#PWR035" (at 142.24 134.62 0)
-      (effects (font (size 1.27 1.27)) hide)
-    )
-    (property "Value" "GND" (at 142.24 133.35 0)
-      (effects (font (size 1.27 1.27)))
-    )
-    (property "Footprint" "" (at 142.24 128.27 0)
-      (effects (font (size 1.27 1.27)) hide)
-    )
-    (property "Datasheet" "" (at 142.24 128.27 0)
-      (effects (font (size 1.27 1.27)) hide)
-    )
-    (pin "1")
-    (instances
-      (project "Pico-Skidi"
-        (path "/21865b85-eb74-4d61-a31a-30858d3bc341/60530e3c-b075-4fd7-83a5-48bc65381cc4"
-          (reference "#PWR035") (unit 1)
-        )
-      )
-    )
-  )
-  (symbol (lib_id "Connector_Generic:Conn_01x03") (at 127 128.27 180) (unit 1)
-    (in_bom yes) (on_board yes) (dnp no) (fields_autoplaced)
-    (property "Reference" "J7" (at 127 119.38 0)
-      (effects (font (size 1.27 1.27)))
-    )
-    (property "Value" "Conn_01x03" (at 127 121.92 0)
-      (effects (font (size 1.27 1.27)))
-    )
-    (property "Footprint" "Connector_PinHeader_2.54mm:PinHeader_1x03_P2.54mm_Vertical" (at 127 128.27 0)
-      (effects (font (size 1.27 1.27)) hide)
-    )
-    (property "Datasheet" "~" (at 127 128.27 0)
-      (effects (font (size 1.27 1.27)) hide)
-    )
-    (pin "1")
-    (pin "2")
-    (pin "3")
-    (instances
-      (project "Pico-Skidi"
-        (path "/21865b85-eb74-4d61-a31a-30858d3bc341/60530e3c-b075-4fd7-83a5-48bc65381cc4"
-          (reference "J7") (unit 1)
-        )
-      )

Commit message: Adding Power
Parts:
- renumbered J8 to J6
Connections:
- no-connect marks 15 -> 14
Changed lines of the file:
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@@
   (junction (at 111.76 97.79) (diameter 0) (color 0 0 0 0)
+  )
+  (junction (at 171.45 69.85) (diameter 0) (color 0 0 0 0)
   )
   (junction (at 111.76 110.49) (diameter 0) (color 0 0 0 0)
@@
   (no_connect (at 144.78 120.65))
   (no_connect (at 139.7 62.23))
-  (no_connect (at 140.97 95.25))
   (no_connect (at 160.02 80.01))
   (no_connect (at 160.02 95.25))
@@
     (stroke (width 0) (type default))
   )
+  (wire (pts (xy 171.45 69.85) (xy 172.72 69.85))
+    (stroke (width 0) (type default))
+  )
   (wire (pts (xy 168.91 110.49) (xy 160.02 110.49))
     (stroke (width 0) (type default))
@@
     (effects (font (size 1.27 1.27)) (justify left))
   )
+  (hierarchical_label "VSYS" (shape input) (at 172.72 69.85 0) (fields_autoplaced)
+    (effects (font (size 1.27 1.27)) (justify left))
+  )
   (hierarchical_label "nFAULT_02" (shape input) (at 124.46 102.87 180) (fields_autoplaced)
     (effects (font (size 1.27 1.27)) (justify right))
@@
   (symbol (lib_id "Connector_Generic:Conn_01x04") (at 200.66 68.58 0) (unit 1)
     (in_bom yes) (on_board yes) (dnp no) (fields_autoplaced)
-    (property "Reference" "J8" (at 203.2 68.58 0)
+    (property "Reference" "J6" (at 203.2 68.58 0)
       (effects (font (size 1.27 1.27)) (justify left))
     )
@@
       (project "Pico-Skidi"
         (path "/21865b85-eb74-4d61-a31a-30858d3bc341/60530e3c-b075-4fd7-83a5-48bc65381cc4"
-          (reference "J8") (unit 1)
+          (reference "J6") (unit 1)
         )
       )
@@
   (symbol (lib_id "power:+3.3V") (at 187.96 68.58 0) (unit 1)
     (in_bom yes) (on_board yes) (dnp no) (fields_autoplaced)
-    (property "Reference" "#PWR040" (at 187.96 72.39 0)
+    (property "Reference" "#PWR026" (at 187.96 72.39 0)
       (effects (font (size 1.27 1.27)) hide)
     )
@@
       (project "Pico-Skidi"
         (path "/21865b85-eb74-4d61-a31a-30858d3bc341/60530e3c-b075-4fd7-83a5-48bc65381cc4"
-          (reference "#PWR040") (unit 1)
+          (reference "#PWR026") (unit 1)
         )
       )
@@
   (symbol (lib_id "power:VBUS") (at 165.1 67.31 0) (unit 1)
     (in_bom yes) (on_board yes) (dnp no) (fields_autoplaced)
-    (property "Reference" "#PWR036" (at 165.1 71.12 0)
+    (property "Reference" "#PWR022" (at 165.1 71.12 0)
       (effects (font (size 1.27 1.27)) hide)
     )
@@
       (project "Pico-Skidi"
         (path "/21865b85-eb74-4d61-a31a-30858d3bc341/60530e3c-b075-4fd7-83a5-48bc65381cc4"
-          (reference "#PWR036") (unit 1)
+          (reference "#PWR022") (unit 1)
         )
       )
@@
   (symbol (lib_id "ExtraPower:VSYS") (at 171.45 69.85 0) (unit 1)
     (in_bom yes) (on_board yes) (dnp no) (fields_autoplaced)
-    (property "Reference" "#PWR05" (at 171.45 73.66 0)
+    (property "Reference" "#PWR025" (at 171.45 73.66 0)
       (effects (font (size 1.27 1.27)) hide)
     )
@@
       (project "Pico-Skidi"
         (path "/21865b85-eb74-4d61-a31a-30858d3bc341/60530e3c-b075-4fd7-83a5-48bc65381cc4"
-          (reference "#PWR05") (unit 1)
+          (reference "#PWR025") (unit 1)
         )
       )
@@
   (symbol (lib_id "power:+3.3V") (at 166.37 78.74 0) (unit 1)
     (in_bom yes) (on_board yes) (dnp no) (fields_autoplaced)
-    (property "Reference" "#PWR037" (at 166.37 82.55 0)
+    (property "Reference" "#PWR023" (at 166.37 82.55 0)
       (effects (font (size 1.27 1.27)) hide)
     )
@@
       (project "Pico-Skidi"
         (path "/21865b85-eb74-4d61-a31a-30858d3bc341/60530e3c-b075-4fd7-83a5-48bc65381cc4"
-          (reference "#PWR037") (unit 1)
+          (reference "#PWR023") (unit 1)
         )
       )
@@
   (symbol (lib_id "power:GND") (at 193.04 62.23 0) (unit 1)
     (in_bom yes) (on_board yes) (dnp no) (fields_autoplaced)
-    (property "Reference" "#PWR041" (at 193.04 68.58 0)
+    (property "Reference" "#PWR027" (at 193.04 68.58 0)
       (effects (font (size 1.27 1.27)) hide)
     )
@@
       (project "Pico-Skidi"
         (path "/21865b85-eb74-4d61-a31a-30858d3bc341/60530e3c-b075-4fd7-83a5-48bc65381cc4"
-          (reference "#PWR041") (unit 1)
+          (reference "#PWR027") (unit 1)
         )
       )
@@
         )
         (path "/21865b85-eb74-4d61-a31a-30858d3bc341/60530e3c-b075-4fd7-83a5-48bc65381cc4"
-          (reference "#PWR038") (unit 1)
+          (reference "#PWR024") (unit 1)
         )
       )
@@
         )
         (path "/21865b85-eb74-4d61-a31a-30858d3bc341/60530e3c-b075-4fd7-83a5-48bc65381cc4"
-          (reference "#PWR034") (unit 1)
-        )
-      )
+          (reference "#PWR021") (unit 1)
+        )
+      )
