File: Servos.kicad_sch (KiCad schematic)
At the start: 2 parts, among them M4 Motor_Servo, M5 Motor_Servo

Commit message: Lots of changes
Parts:
- added M4 (x2), M5 (x2): Motor_Servo, symbol Motor:Motor_Servo
- M4: footprint (none) -> Connector_PinHeader_2.54mm:PinHeader_1x03_P2.54mm_Vertical
Connections:
- net GND: now also M4.3 (-), M4.3 (-), M5.3 (-), M5.3 (-)
- net SRV_01: now reaches M4.1 (PWM)
- net +5V: now reaches M4.2 (+)
- net +5V: now also M5.2 (+), M4.2 (+), M4.2 (+), M5.2 (+), M5.2 (+)
- net SRV_02: now reaches M5.1 (PWM)
- new net SRV_03: M4.1 (PWM)
- new net SRV_04: M5.1 (PWM)
- new net SRV_05: M4.1 (PWM)
- new net SRV_06: M5.1 (PWM)
Other:
- moved on the sheet: M4, M5

Commit message: syncing
Parts:
- M4, M5: footprint (none) -> Connector_PinHeader_2.54mm:PinHeader_1x03_P2.54mm_Vertical
